File: stensgrind_pcb/stensgrind_pcb.kicad_pcb (KiCad board)
At the start: 4 copper layers, 158.9 x 99.5 mm, 84 parts, among them J1 Conn_01x04_Pin, J2 SERIAL_01, J3 DISPLAY_01, SW1 SW_PUSH, SW10 SW_PUSH, SW11 SW_PUSH, SW12 SW_PUSH, SW13 SW_PUSH, SW14 SW_PUSH, SW15 SW_PUSH, SW16 SW_PUSH, SW17 SW_PUSH, SW18 SW_PUSH, SW19 SW_PUSH, SW2 SW_PUSH, SW20 SW_PUSH, SW21 SW_PUSH, SW22 SW_PUSH, SW23 SW_PUSH, SW3 SW_PUSH, SW4 SW_PUSH, SW5 SW_PUSH, SW6 SW_PUSH, SW7 SW_PUSH, SW8 SW_PUSH, SW9 SW_PUSH, U1 ProMicro_r, U10 4492, U11 4492, U12 4492, U13 4492, U14 4492, U15 4492, U16 4492, U17 4492, U18 4492, U19 4492, U2 CAHCT1G125QDCKRQ1, U20 4492, U21 4492, U22 4492, U23 4492, U24 4492, U25 4492, U26 ISO1050DUB, U3 4492, U4 4492, U5 4492, U6 4492, U7 4492, U8 4492, U9 4492

Commit message: Add link to project
Other:
- board text added: "https://github.com/Deltaphish/stensgrind"
Changed lines of the file:
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@@
+		)
+	)
+	(gr_text "https://github.com/Deltaphish/stensgrind"
+		(at 192.4 71.1 90)
+		(layer "B.SilkS")
+		(effects
+			(font
+				(size 1 1)
+				(thickness 0.1)
+			)
+			(justify left bottom mirror)
 		)
 	)

Commit message: add right half
Parts:
- added /RIGHT_SIDE/COL5: , PAD_0_5MM, F.Cu at (245.5, 151.5)
- added C3: 0.1uf, Capacitor_SMD:C_0805_2012Metric_Pad1.18x1.45mm_HandSolder, F.Cu at (333.0, 165.3)
- added C4: 0.1uf, Capacitor_SMD:C_0805_2012Metric_Pad1.18x1.45mm_HandSolder, F.Cu at (339.5, 165.3)
- added COL1: , PAD_0_5MM, F.Cu at (245.5, 162.7)
- added COL10: , PAD_0_5MM, F.Cu at (245.5, 137.5)
- added COL11: , PAD_0_5MM, F.Cu at (245.5, 134.7)
- added COL12: , PAD_0_5MM, F.Cu at (245.5, 131.9)
- added COL13: , PAD_0_5MM, F.Cu at (245.5, 129.1)
- added COL14: , PAD_0_5MM, F.Cu at (245.5, 126.3)
- added COL15: , PAD_0_5MM, F.Cu at (245.5, 123.5)
- added COL16: , PAD_0_5MM, F.Cu at (245.5, 120.7)
- added COL17: , PAD_0_5MM, F.Cu at (245.5, 117.9)
- added COL18: , PAD_0_5MM, F.Cu at (245.5, 115.1)
- added COL19: , PAD_0_5MM, F.Cu at (245.5, 112.3)
- added COL2: , PAD_0_5MM, F.Cu at (245.5, 159.9)
- added COL20: , PAD_0_5MM, F.Cu at (245.5, 109.5)
- added COL3: , PAD_0_5MM, F.Cu at (245.5, 157.1)
- added COL4: , PAD_0_5MM, F.Cu at (245.5, 154.3)
- added COL6: , PAD_0_5MM, F.Cu at (245.5, 148.7)
- added COL7: , PAD_0_5MM, F.Cu at (245.5, 145.9)
- added COL8: , PAD_0_5MM, F.Cu at (245.5, 143.1)
- added COL9: , PAD_0_5MM, F.Cu at (245.5, 140.3)
- added D24: D, Diode_THT:D_DO-35_SOD27_P10.16mm_Horizontal, B.Cu at (365.9, 127.3)
- added D25: D, Diode_THT:D_DO-35_SOD27_P10.16mm_Horizontal, B.Cu at (365.9, 146.3)
- added D26: D, Diode_THT:D_DO-35_SOD27_P10.16mm_Horizontal, B.Cu at (365.9, 165.5)
- added D27: D, Diode_THT:D_DO-35_SOD27_P10.16mm_Horizontal, B.Cu at (279.4, 165.3)
- added D28: D, Diode_THT:D_DO-35_SOD27_P10.16mm_Horizontal, B.Cu at (361.5, 161.1)
- added D29: D, Diode_THT:D_DO-35_SOD27_P10.16mm_Horizontal, B.Cu at (260.4, 165.8)
- added D30: D, Diode_THT:D_DO-35_SOD27_P10.16mm_Horizontal, B.Cu at (346.7, 146.3)
- added D31: D, Diode_THT:D_DO-35_SOD27_P10.16mm_Horizontal, B.Cu at (346.7, 127.1)
- added D32: D, Diode_THT:D_DO-35_SOD27_P10.16mm_Horizontal, B.Cu at (327.5, 160.8)
- added D33: D, Diode_THT:D_DO-35_SOD27_P10.16mm_Horizontal, B.Cu at (241.4, 166.3)
- added D34: D, Diode_THT:D_DO-35_SOD27_P10.16mm_Horizontal, B.Cu at (327.5, 141.7)
- added D35: D, Diode_THT:D_DO-35_SOD27_P10.16mm_Horizontal, B.Cu at (327.5, 122.5)
- added D36: D, Diode_THT:D_DO-35_SOD27_P10.16mm_Horizontal, B.Cu at (322.0, 154.4)
- added D37: D, Diode_THT:D_DO-35_SOD27_P10.16mm_Horizontal, B.Cu at (250.7, 146.3)
- added D38: D, Diode_THT:D_DO-35_SOD27_P10.16mm_Horizontal, B.Cu at (308.3, 139.3)
- added D39: D, Diode_THT:D_DO-35_SOD27_P10.16mm_Horizontal, B.Cu at (308.3, 120.0)
- added D40: D, Diode_THT:D_DO-35_SOD27_P10.16mm_Horizontal, B.Cu at (303.5, 156.3)
- added D41: D, Diode_THT:D_DO-35_SOD27_P10.16mm_Horizontal, B.Cu at (250.7, 127.3)
- added D42: D, Diode_THT:D_DO-35_SOD27_P10.16mm_Horizontal, B.Cu at (289.1, 141.7)
- added D43: D, Diode_THT:D_DO-35_SOD27_P10.16mm_Horizontal, B.Cu at (289.1, 122.4)
- added D44: D, Diode_THT:D_DO-35_SOD27_P10.16mm_Horizontal, B.Cu at (269.9, 124.8)
- added D45: D, Diode_THT:D_DO-35_SOD27_P10.16mm_Horizontal, B.Cu at (269.9, 144.0)
- added D46: D, Diode_THT:D_DO-35_SOD27_P10.16mm_Horizontal, B.Cu at (284.0, 158.9)
- added J5: SERIAL_01, Connector_PinSocket_2.54mm:PinSocket_1x03_P2.54mm_Vertical, F.Cu at (340.5, 178.8)
- added J6: Conn_01x04_Pin, Connector_PinSocket_2.54mm:PinSocket_1x04_P2.54mm_Vertical, F.Cu at (348.0, 175.1)
- added R10: 100k, Resistor_SMD:R_1206_3216Metric_Pad1.30x1.75mm_HandSolder, F.Cu at (305.0, 174.8)
- added R4: 100k, Resistor_SMD:R_1206_3216Metric_Pad1.30x1.75mm_HandSolder, F.Cu at (297.5, 174.8)
- added R7: 120, Resistor_SMD:R_1206_3216Metric_Pad1.30x1.75mm_HandSolder, F.Cu at (351.5, 171.6)
- added R8: 100k, Resistor_SMD:R_1206_3216Metric_Pad1.30x1.75mm_HandSolder, F.Cu at (300.0, 174.8)
- added R9: 100k, Resistor_SMD:R_1206_3216Metric_Pad1.30x1.75mm_HandSolder, F.Cu at (302.5, 174.8)
- added ROW1: , PAD_0_5MM, F.Cu at (244.8, 163.7)
- added ROW10: , PAD_0_5MM, F.Cu at (226.1, 163.7)
- added ROW11: , PAD_0_5MM, F.Cu at (224.1, 163.7)
- added ROW12: , PAD_0_5MM, F.Cu at (222.0, 163.7)
- added ROW13: , PAD_0_5MM, F.Cu at (219.9, 163.7)
- added ROW14: , PAD_0_5MM, F.Cu at (217.9, 163.7)
- added ROW2: , PAD_0_5MM, F.Cu at (242.7, 163.7)
- added ROW3: , PAD_0_5MM, F.Cu at (240.6, 163.7)
- added ROW4: , PAD_0_5MM, F.Cu at (238.6, 163.7)
- added ROW5: , PAD_0_5MM, F.Cu at (236.5, 163.7)
- added ROW6: , PAD_0_5MM, F.Cu at (234.4, 163.7)
- added ROW7: , PAD_0_5MM, F.Cu at (232.4, 163.7)
- added ROW8: , PAD_0_5MM, F.Cu at (230.3, 163.7)
- added ROW9: , PAD_0_5MM, F.Cu at (228.2, 163.7)
- added R_LED_DATA_3: 500, Resistor_SMD:R_1206_3216Metric_Pad1.30x1.75mm_HandSolder, F.Cu at (158.6, 155.5)
- added R_LED_DATA_4: 500, Resistor_SMD:R_1206_3216Metric_Pad1.30x1.75mm_HandSolder, F.Cu at (165.6, 112.2)
- added SW24: SW_PUSH, kbd:keyswitch_cherrymx_hotswap_1u, B.Cu at (371.0, 117.6)
- added SW25: SW_PUSH, kbd:keyswitch_cherrymx_hotswap_1u, B.Cu at (371.0, 136.8)
- added SW26: SW_PUSH, kbd:keyswitch_cherrymx_hotswap_1u, B.Cu at (371.0, 156.0)
- added SW27: SW_PUSH, kbd:keyswitch_cherrymx_hotswap_1u, B.Cu at (284.6, 175.2)
- added SW28: SW_PUSH, kbd:keyswitch_cherrymx_hotswap_1u, B.Cu at (351.8, 117.6)
- added SW29: SW_PUSH, kbd:keyswitch_cherrymx_hotswap_1u, B.Cu at (351.8, 136.8)
- added SW30: SW_PUSH, kbd:keyswitch_cherrymx_hotswap_1u, B.Cu at (351.8, 156.0)
- added SW31: SW_PUSH, kbd:keyswitch_cherrymx_hotswap_1u, B.Cu at (265.5, 175.3)
- added SW32: SW_PUSH, kbd:keyswitch_cherrymx_hotswap_1u, B.Cu at (332.6, 112.9)
- added SW33: SW_PUSH, kbd:keyswitch_cherrymx_hotswap_1u, B.Cu at (332.6, 132.1)
- added SW34: SW_PUSH, kbd:keyswitch_cherrymx_hotswap_1u, B.Cu at (332.6, 151.3)
- added SW35: SW_PUSH, kbd:keyswitch_cherrymx_hotswap_1u, B.Cu at (246.4, 175.3)
- added SW36: SW_PUSH, kbd:keyswitch_cherrymx_hotswap_1u, B.Cu at (313.4, 110.5)
- added SW37: SW_PUSH, kbd:keyswitch_cherrymx_hotswap_1u, B.Cu at (313.4, 129.7)
- added SW38: SW_PUSH, kbd:keyswitch_cherrymx_hotswap_1u, B.Cu at (313.4, 148.9)
- added SW39: SW_PUSH, kbd:keyswitch_cherrymx_hotswap_1u, B.Cu at (255.8, 136.8)
- added SW40: SW_PUSH, kbd:keyswitch_cherrymx_hotswap_1u, B.Cu at (294.2, 112.9)
- added SW41: SW_PUSH, kbd:keyswitch_cherrymx_hotswap_1u, B.Cu at (294.2, 132.1)
- added SW42: SW_PUSH, kbd:keyswitch_cherrymx_hotswap_1u, B.Cu at (294.2, 151.3)
- added SW43: SW_PUSH, kbd:keyswitch_cherrymx_hotswap_1u, B.Cu at (255.8, 117.6)
- added SW44: SW_PUSH, kbd:keyswitch_cherrymx_hotswap_1u, B.Cu at (275.0, 115.2)
- added SW45: SW_PUSH, kbd:keyswitch_cherrymx_hotswap_1u, B.Cu at (275.0, 134.4)
- added SW46: SW_PUSH, kbd:keyswitch_cherrymx_hotswap_1u, B.Cu at (275.0, 153.6)
- added TOUCH_COL1: TESTPOINTPAD_0_5MM, TestPoint:TestPoint_Pad_D1.0mm, F.Cu at (249.0, 152.0)
- added TOUCH_COL5: TESTPOINTPAD_0_5MM, TestPoint:TestPoint_Pad_D1.0mm, F.Cu at (248.0, 149.5)
- added U27: ProMicro_r, kbd:ProMicro, B.Cu at (310.5, 171.3)
- added U28: ISO1050DUB, Package_SO:SOP-8_6.62x9.15mm_P2.54mm, F.Cu at (338.5, 171.3)
- added U29: CAHCT1G125QDCKRQ1, DEV_18288:DCK5, F.Cu at (309.9, 174.3)
- added U30: 4492, DEV_18288:LED_4492, F.Cu at (332.5, 155.8)
- added U31: 4492, DEV_18288:LED_4492, F.Cu at (352.0, 160.8)
- added U32: 4492, DEV_18288:LED_4492, F.Cu at (371.0, 160.8)
- added U33: 4492, DEV_18288:LED_4492, F.Cu at (371.0, 141.3)
- added U34: 4492, DEV_18288:LED_4492, F.Cu at (371.0, 122.3)
- added U35: 4492, DEV_18288:LED_4492, F.Cu at (351.5, 122.3)
- added U36: 4492, DEV_18288:LED_4492, F.Cu at (352.0, 141.8)
- added U37: 4492, DEV_18288:LED_4492, F.Cu at (332.5, 136.8)
- added U38: 4492, DEV_18288:LED_4492, F.Cu at (332.5, 117.8)
- added U39: 4492, DEV_18288:LED_4492, F.Cu at (313.5, 115.3)
- added U40: 4492, DEV_18288:LED_4492, F.Cu at (313.5, 134.3)
- added U41: 4492, DEV_18288:LED_4492, F.Cu at (294.0, 136.8)
- added U42: 4492, DEV_18288:LED_4492, F.Cu at (294.0, 117.8)
- added U43: 4492, DEV_18288:LED_4492, F.Cu at (275.0, 119.8)
- added U44: 4492, DEV_18288:LED_4492, F.Cu at (275.0, 139.3)
- added U45: 4492, DEV_18288:LED_4492, F.Cu at (255.5, 122.3)
- added U46: 4492, DEV_18288:LED_4492, F.Cu at (255.5, 141.8)
- added U47: 4492, DEV_18288:LED_4492, F.Cu at (275.0, 158.3)
- added U48: 4492, DEV_18288:LED_4492, F.Cu at (246.5, 180.3)
- added U49: 4492, DEV_18288:LED_4492, F.Cu at (265.5, 180.3)
- added U50: 4492, DEV_18288:LED_4492, F.Cu at (284.5, 179.8)
- added U51: 4492, DEV_18288:LED_4492, F.Cu at (294.5, 155.8)
- added U52: 4492, DEV_18288:LED_4492, F.Cu at (313.5, 153.8)
- added U53: ~, Package_DFN_QFN:IQS9150, F.Cu at (256.6, 156.2)
- moved R_LED_DATA_1 180.4 mm to (319.0, 160.3)
- moved R_LED_DATA_2 162.8 mm to (312.0, 170.8), turned to 180 degrees
- moved U1 50.7 mm to (178.2, 130.7)
- moved C1 50.7 mm to (171.8, 157.9)
- moved J3 50.7 mm to (183.4, 158.9)
- moved R6 50.7 mm to (174.1, 144.1)
- moved U2 50.7 mm to (173.0, 117.6)
- moved J2 50.7 mm to (188.9, 111.2)
- moved C2 50.7 mm to (186.5, 155.5)
- moved J1 50.7 mm to (171.6, 147.4)
- moved R1 50.7 mm to (174.1, 136.4)
- moved R2 50.7 mm to (174.1, 138.9)
- moved R3 50.7 mm to (167.8, 154.6)
- moved R5 50.7 mm to (174.1, 141.4)
- moved U26 50.7 mm to (179.5, 152.1)
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Connections:
- net /CAN+ renamed /LEFT_SIDE/CAN+
- net /CAN- renamed /LEFT_SIDE/CAN-
- net CAN_RX renamed /LEFT_SIDE/CAN_RX
- net CAN_TX renamed /LEFT_SIDE/CAN_TX
- net COL_1 renamed /LEFT_SIDE/COL_1
- net COL_2 renamed /LEFT_SIDE/COL_2
- net COL_3 renamed /LEFT_SIDE/COL_3
- net COL_4 renamed /LEFT_SIDE/COL_4
- net COL_5 renamed /LEFT_SIDE/COL_5
- net COL_6 renamed /LEFT_SIDE/COL_6
- net LED_DOUT_V3.3 renamed /LEFT_SIDE/LED_DOUT_V3.3
- net ROW_1 renamed /LEFT_SIDE/ROW_1
- net ROW_2 renamed /LEFT_SIDE/ROW_2
- net ROW_3 renamed /LEFT_SIDE/ROW_3
- net ROW_4 renamed /LEFT_SIDE/ROW_4
- net SCL renamed /LEFT_SIDE/SCL
- net SDA renamed /LEFT_SIDE/SDA
- net SERIAL_RX renamed /LEFT_SIDE/SERIAL_RX
- net SERIAL_TX renamed /LEFT_SIDE/SERIAL_TX
- net V3.3 renamed /LEFT_SIDE/V3.3
- net V5 renamed /LEFT_SIDE/V5
- C1 pad 1: GNDR -> GNDL
- C2 pad 1: GNDR -> GNDL
- J1 pad 1: GNDR -> GNDL
- J2 pad 1: GNDR -> GNDL
- J3 pad 1: GNDR -> GNDL
- R1 pad 2: GNDR -> GNDL
- R2 pad 2: GNDR -> GNDL
- R5 pad 2: GNDR -> GNDL
- R6 pad 2: GNDR -> GNDL
- R_LED_DATA_1 pad 1: Net-(U3-DIN) -> Net-(U52-DOUT)
- R_LED_DATA_1 pad 2: LED_DOUT_V5 -> GNDR
- R_LED_DATA_2 pad 1: Net-(U25-DOUT) -> Net-(U30-DIN)
- R_LED_DATA_2 pad 2: GNDR -> /RIGHT_SIDE/LED_DOUT_V5
- U1 pad 17: unconnected-(U1-A0/F7-Pad17) -> /LEFT_SIDE/NC
- U1 pad 22: unconnected-(U1-RST-Pad22) -> /LEFT_SIDE/RST
- U1 pad 23: GNDR -> GNDL
- U1 pad 3: GNDR -> GNDL
- U1 pad 4: GNDR -> GNDL
- U10 pad 4: GNDR -> GNDL
- U11 pad 4: GNDR -> GNDL
- U12 pad 4: GNDR -> GNDL
- U13 pad 4: GNDR -> GNDL
- U14 pad 4: GNDR -> GNDL
- U15 pad 4: GNDR -> GNDL
- U16 pad 4: GNDR -> GNDL
- U17 pad 4: GNDR -> GNDL
- U18 pad 4: GNDR -> GNDL
- U19 pad 4: GNDR -> GNDL
- U2 pad 1: GNDR -> GNDL
- U2 pad 3: GNDR -> GNDL
- U2 pad 4: LED_DOUT_V5 -> /LEFT_SIDE/LED_DOUT_V5
- U20 pad 4: GNDR -> GNDL
- U21 pad 4: GNDR -> GNDL
- U22 pad 4: GNDR -> GNDL
- U23 pad 4: GNDR -> GNDL
- U24 pad 4: GNDR -> GNDL
- U25 pad 4: GNDR -> GNDL
- U26 pad 4: GNDR -> GNDL
- U26 pad 5: GNDR -> GNDL
- U3 pad 4: GNDR -> GNDL
- U4 pad 4: GNDR -> GNDL
- U5 pad 4: GNDR -> GNDL
- U6 pad 4: GNDR -> GNDL
- U7 pad 4: GNDR -> GNDL
- U8 pad 4: GNDR -> GNDL
- U9 pad 4: GNDR -> GNDL
Routing:
- net /RIGHT_SIDE/ROW_2: track 0.00 -> 178.5 mm
- net /RIGHT_SIDE/ROW_3: track 0.00 -> 160.8 mm
- net /RIGHT_SIDE/ROW_1: track 0.00 -> 160.4 mm, vias 0 -> 2
- net /RIGHT_SIDE/COL_2: track 0.00 -> 146.4 mm, vias 0 -> 1
- net /RIGHT_SIDE/COL_1: track 0.00 -> 137.8 mm
- net /RIGHT_SIDE/COL_3: track 0.00 -> 137.0 mm, vias 0 -> 1
- net /RIGHT_SIDE/ROW_4: track 0.00 -> 125.2 mm
- net /RIGHT_SIDE/COL_5: track 0.00 -> 100.6 mm
- net /RIGHT_SIDE/COL_6: track 0.00 -> 74.1 mm
- net /LEFT_SIDE/COL_3: track 283.3 -> 216.6 mm
- net GNDR: track 61.3 -> 0.00 mm, vias 31 -> 0
- net /LEFT_SIDE/COL_6: track 121.1 -> 60.3 mm
- net /RIGHT_SIDE/SERIAL_RX: track 0.00 -> 58.3 mm
- net GNDL: track 0.00 -> 58.2 mm, vias 0 -> 24
- net /RIGHT_SIDE/COL_4: track 0.00 -> 57.5 mm
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- added copper zone on In2.Cu, net /RIGHT_SIDE/V5
- added copper zone on F.Cu, net COL1
- added copper zone on F.Cu, net COL10
- added copper zone on F.Cu, net COL11
- added copper zone on F.Cu, net COL12
- added copper zone on F.Cu, net COL13
- added copper zone on F.Cu, net COL14
- added copper zone on F.Cu, net COL15
- added copper zone on F.Cu, net COL16
- added copper zone on F.Cu, net COL17
- added copper zone on F.Cu, net COL18
- added copper zone on F.Cu, net COL19
- added copper zone on F.Cu, net COL2
- added copper zone on F.Cu, net COL20
- added copper zone on F.Cu, net COL3
- added copper zone on F.Cu, net COL4
- added copper zone on F.Cu, net COL5
- added copper zone on F.Cu, net COL6
- added copper zone on F.Cu, net COL7
- added copper zone on F.Cu, net COL8
- added copper zone on F.Cu, net COL9
- added copper zone on In1.Cu, net GNDL
- added copper zone on F.Cu, net ROW1
- added copper zone on F.Cu, net ROW10
- added copper zone on F.Cu, net ROW11
- added copper zone on F.Cu, net ROW12
- added copper zone on F.Cu, net ROW13
- added copper zone on F.Cu, net ROW14
- added copper zone on F.Cu, net ROW2
- added copper zone on F.Cu, net ROW3
- added copper zone on F.Cu, net ROW4
- added copper zone on F.Cu, net ROW5
- added copper zone on F.Cu, net ROW6
- added copper zone on F.Cu, net ROW7
- added copper zone on F.Cu, net ROW8
- added copper zone on F.Cu, net ROW9
Other:
- board size 158.9 x 99.5 mm -> 349.9 x 99.5 mm
- board text added: "STENSGRIND V1.0 R"
