File: stensgrind_pcb/stensgrind_pcb.kicad_pcb (KiCad board)
At the start: 4 copper layers, 352 x 100.1 mm, 177 parts, among them J1 Conn_01x04_Pin, J2 SERIAL_01, J3 DISPLAY_01, J4 Conn_01x04_Pin, J5 SERIAL_01, J6 Conn_01x04_Pin, SW1 SW_PUSH, SW10 SW_PUSH, SW11 SW_PUSH, SW12 SW_PUSH, SW13 SW_PUSH, SW14 SW_PUSH, SW15 SW_PUSH, SW16 SW_PUSH, SW17 SW_PUSH, SW18 SW_PUSH, SW19 SW_PUSH, SW2 SW_PUSH, SW20 SW_PUSH, SW21 SW_PUSH, SW22 SW_PUSH, SW23 SW_PUSH, SW24 SW_PUSH, SW25 SW_PUSH, SW26 SW_PUSH, SW27 SW_PUSH, SW28 SW_PUSH, SW29 SW_PUSH, SW3 SW_PUSH, SW30 SW_PUSH, SW31 SW_PUSH, SW32 SW_PUSH, SW33 SW_PUSH, SW34 SW_PUSH, SW35 SW_PUSH, SW36 SW_PUSH, SW37 SW_PUSH, SW38 SW_PUSH, SW39 SW_PUSH, SW4 SW_PUSH, SW40 SW_PUSH, SW41 SW_PUSH, SW42 SW_PUSH, SW43 SW_PUSH, SW44 SW_PUSH, SW45 SW_PUSH, SW46 SW_PUSH, SW5 SW_PUSH, SW6 SW_PUSH, SW7 SW_PUSH, SW8 SW_PUSH, SW9 SW_PUSH, U1 ProMicro_r, U10 4492, U11 4492, U12 4492, U13 4492, U14 4492, U15 4492, U16 4492, U17 4492, U18 4492, U19 4492, U2 CAHCT1G125QDCKRQ1, U20 4492, U21 4492, U22 4492, U23 4492, U24 4492, U25 4492, U26 ISO1050DUB, U27 ProMicro_r, U28 ISO1050DUB, U29 CAHCT1G125QDCKRQ1, U3 4492, U30 4492, U31 4492, U32 4492, U33 4492, U34 4492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

Commit message: finish up v1
Parts:
- added D47: LED, LED_SMD:LED_1206_3216Metric, F.Cu at (248.0, 168.5)
- added LEFT: Board, PCM_kikit:Board, F.Cu at (31.7, 103.8)
- added MNT 1: MountingHole_3.2mm_M3, MountingHole:MountingHole_3.2mm_M3, F.Cu at (150.0, 189.0)
- added MNT 2: MountingHole_3.2mm_M3, MountingHole:MountingHole_3.2mm_M3, F.Cu at (99.5, 159.0)
- added MNT 3: MountingHole_2.2mm_M2, MountingHole:MountingHole_2.2mm_M2, F.Cu at (149.5, 105.0)
- added MNT 4: MountingHole_2.2mm_M2, MountingHole:MountingHole_2.2mm_M2, F.Cu at (67.5, 102.0)
- added R11: R, Resistor_SMD:R_1206_3216Metric_Pad1.30x1.75mm_HandSolder, F.Cu at (252.4, 169.5)
- added RIGHT: Board, PCM_kikit:Board, F.Cu at (227.5, 115.5)
- added TP3: 0.5mm, PCM_SparkFun-Connector:TestPoint-0.5mm, F.Cu at (250.5, 166.5)
- moved U21 65.6 mm to (118.2, 114.3), turned to 0 degrees
- moved U5 65.6 mm to (128.6, 179.1), turned to -11.94 degrees
- moved U6 65.6 mm to (108.3, 176.9)
- moved U22 64.0 mm to (137.4, 116.9), turned to 0 degrees
- moved U4 64.0 mm to (155.9, 178.2), turned to -23.88 degrees
- moved U7 54.4 mm to (118.0, 153.0)
- moved U9 51.0 mm to (79.8, 152.9)
- moved U8 49.5 mm to (98.8, 150.6)
- moved U20 44.4 mm to (118.2, 133.6)
- moved R_LED_DATA_4 43.2 mm to (154.5, 154.0)
- moved C2 38.5 mm to (170.5, 120.5)
- moved C1 38.0 mm to (178.5, 120.5), turned to -90 degrees
- moved U3 34.9 mm to (137.2, 155.2)
- moved U2 32.2 mm to (168.9, 149.5)
- moved U18 28.8 mm to (99.1, 112.0)
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Connections:
- U1 pad 18: /LEFT_SIDE/CAN_TX -> /LEFT_SIDE/LED_DOUT_V3.3
- U1 pad 19: /LEFT_SIDE/CAN_RX -> /LEFT_SIDE/CAN_TX
- U1 pad 20: /LEFT_SIDE/LED_DOUT_V3.3 -> /LEFT_SIDE/CAN_RX
- U1 pad 7: /LEFT_SIDE/COL_5 -> /LEFT_SIDE/COL_6
- U1 pad 8: /LEFT_SIDE/COL_6 -> /LEFT_SIDE/COL_4
- U1 pad 9: /LEFT_SIDE/COL_4 -> /LEFT_SIDE/COL_5
- U27 pad 8: /RIGHT_SIDE/NC -> /RIGHT_SIDE/STATUS_LED
Routing:
- net /LEFT_SIDE/COL_3: track 0.00 -> 269.8 mm
- net /LEFT_SIDE/COL_1: track 0.00 -> 243.1 mm
- net /LEFT_SIDE/COL_2: track 0.00 -> 215.7 mm, vias 0 -> 2
- net /LEFT_SIDE/COL_4: track 0.00 -> 195.7 mm
- net /LEFT_SIDE/ROW_1: track 0.00 -> 161.6 mm
- net /LEFT_SIDE/COL_5: track 0.00 -> 148.4 mm
- net /LEFT_SIDE/ROW_2: track 0.00 -> 132.1 mm
- net /LEFT_SIDE/ROW_3: track 0.00 -> 129.8 mm
- net /LEFT_SIDE/COL_6: track 0.00 -> 114.7 mm, vias 0 -> 2
- net /LEFT_SIDE/ROW_4: track 0.00 -> 97.2 mm
- net GNDL: track 0.00 -> 69.3 mm, vias 0 -> 27
- net /LEFT_SIDE/V5: track 0.00 -> 49.2 mm, vias 0 -> 25
- net /RIGHT_SIDE/STATUS_LED: track 0.00 -> 42.8 mm
- net Net-(U6-DOUT): track 0.00 -> 38.4 mm
- net GNDR: track 26.2 -> 63.7 mm, vias 5 -> 30
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Other:
- board size 352 x 100.1 mm -> 351.8 x 100.3 mm

Commit message: fix i2c mapping
Parts:
- moved J4 7.62 mm to (230.0, 155.0), turned to 90 degrees
- moved J3 7.52 mm to (180.5, 151.5), turned to -90 degrees
Connections:
- J4 pad 1: /RIGHT_SIDE/SCL -> /RIGHT_SIDE/SDA
- J4 pad 2: /RIGHT_SIDE/SDA -> /RIGHT_SIDE/SCL
Routing:
- net /LEFT_SIDE/SDA: track 28.1 -> 39.7 mm
- net /RIGHT_SIDE/SCL: track 29.4 -> 34.4 mm
- net /RIGHT_SIDE/SDA: track 32.0 -> 36.1 mm
- net /LEFT_SIDE/SCL: track 26.8 -> 29.5 mm
