File: stensgrind_pcb/left.kicad_sch (KiCad schematic)
At the start: 84 parts, among them J1 Conn_01x04_Pin, J2 SERIAL_01, J3 DISPLAY_01, SW1 SW_PUSH, SW10 SW_PUSH, SW11 SW_PUSH, SW12 SW_PUSH, SW13 SW_PUSH, SW14 SW_PUSH, SW15 SW_PUSH, SW16 SW_PUSH, SW17 SW_PUSH, SW18 SW_PUSH, SW19 SW_PUSH, SW2 SW_PUSH, SW20 SW_PUSH, SW21 SW_PUSH, SW22 SW_PUSH, SW23 SW_PUSH, SW3 SW_PUSH, SW4 SW_PUSH, SW5 SW_PUSH, SW6 SW_PUSH, SW7 SW_PUSH, SW8 SW_PUSH, SW9 SW_PUSH, U1 ProMicro_r, U10 4492, U11 4492, U12 4492, U13 4492, U14 4492, U15 4492, U16 4492, U17 4492, U18 4492, U19 4492, U2 CAHCT1G125QDCKRQ1, U20 4492, U21 4492, U22 4492, U23 4492, U24 4492, U25 4492, U26 ISO1050DUB, U3 4492, U4 4492, U5 4492, U6 4492, U7 4492, U8 4492, U9 4492

Commit message: finish up v1
Connections:
- net CAN_RX: now also U1.20 (A3/F4); no longer U1.19 (A2/F5)
- net CAN_TX: now also U1.19 (A2/F5); no longer U1.18 (A1/F6)
- net COL_4: now also U1.8 (C6/5); no longer U1.9 (D7/6)
- net COL_5: now also U1.9 (D7/6); no longer U1.7 (D4/4)
- net COL_6: now also U1.7 (D4/4); no longer U1.8 (C6/5)
- net LED_DOUT_V3.3: now also U1.18 (A1/F6); no longer U1.20 (A3/F4)
